File: board.kicad_pcb (KiCad board)
At the start: 2 copper layers, 100 x 100 mm, 70 parts, among them J1 JST_XH_LED_POWER, J2 JST-XH_LED, U1 LM3414, U2 LM3414, U3 LM3414

Commit message: Syncing AISLER project with GitHub repository
Parts:
- removed JP1, JP2, JP3: Current mesurment, Connector_PinHeader_2.54mm:PinHeader_1x02_P2.54mm_Vertical
- removed the REF** at (66.7, 130.8)
- removed RV1, RV2, RV3: 5k, footprints:ST4ETA502
- removed TP10: GND, Connector_PinHeader_2.54mm:PinHeader_1x01_P2.54mm_Vertical
- TP2: value Red -> Test_Point; footprint Connector_PinHeader_2.54mm:PinHeader_1x01_P2.54mm_Vertical -> TestPoint:TestPoint_Pad_D2.0mm
- TP4: value Blue -> Test_Point; footprint Connector_PinHeader_2.54mm:PinHeader_1x01_P2.54mm_Vertical -> TestPoint:TestPoint_Pad_D2.0mm
- TP5: value +24V -> Test_Point; footprint Connector_PinHeader_2.54mm:PinHeader_1x01_P2.54mm_Vertical -> TestPoint:TestPoint_Pad_D2.0mm
- TP6: value Far -> Test_Point; footprint Connector_PinHeader_2.54mm:PinHeader_1x01_P2.54mm_Vertical -> TestPoint:TestPoint_Pad_D2.0mm
- moved TP2 26.9 mm to (109.5, 129.2)
- moved TP4 9.86 mm to (96.8, 130.0)
- moved TP6 8.82 mm to (101.8, 130.0)
- moved G*** 8.03 mm to (67.5, 84.8)
- moved R5 7.21 mm to (131.2, 120.5), turned to 147.7 degrees
- moved R1 6.62 mm to (106.8, 62.8), turned to 257.3 degrees
- moved REF** 3.20 mm to (99.5, 138.4)
- moved C1 2.51 mm to (107.8, 58.2), turned to 257.3 degrees
- moved G*** 2.27 mm to (136.5, 111.5)
- moved R3 2.27 mm to (56.8, 91.0), turned to 167.3 degrees
- moved TP5 1.97 mm to (73.0, 113.8), turned to 270 degrees
- turned C4 to 327.7 degrees
Connections:
- L2 pad 1: Net-(JP2-Pad2) -> Net-(D15-Pad1)
- L3 pad 1: Net-(JP3-Pad2) -> Net-(D19-Pad1)
- R9 pad 1: Net-(JP1-Pad2) -> Net-(D9-Pad1)
- TP2 pad 1: Net-(JP1-Pad2) -> Net-(D9-Pad1)
- TP4 pad 1: Net-(JP2-Pad2) -> Net-(D15-Pad1)
- TP6 pad 1: Net-(JP3-Pad2) -> Net-(D19-Pad1)
- U1 pad 3: Net-(RV1-Pad2) -> Net-(R1-Pad1)
- U2 pad 3: Net-(RV2-Pad2) -> Net-(R3-Pad1)
- U3 pad 3: Net-(RV3-Pad2) -> Net-(R5-Pad1)
Routing:
- net Net-(JP3-Pad2): track 21.8 -> 0.00 mm
- net Net-(D9-Pad1): track 26.9 -> 43.3 mm
- net Net-(JP2-Pad2): track 15.4 -> 0.00 mm
- net Net-(D19-Pad1): track 17.9 -> 32.9 mm
- net Net-(D15-Pad1): track 43.2 -> 58.1 mm
- net Net-(JP1-Pad2): track 14.4 -> 0.00 mm
- net Net-(RV2-Pad2): track 10.3 -> 0.00 mm
- net Net-(RV1-Pad2): track 6.47 -> 0.00 mm
- net Net-(RV3-Pad2): track 5.68 -> 0.00 mm
- net +24V: track 324.4 -> 320.3 mm
- net Net-(C1-Pad1): track 3.35 -> 6.22 mm
- net Net-(R1-Pad1): track 3.61 -> 5.61 mm
- net Net-(R5-Pad1): track 4.66 -> 5.84 mm
- net Net-(C4-Pad1): track 5.49 -> 6.14 mm
Other:
- board text added: "R_IADJ"
- board text removed: "+Blue-"
- board text removed: "+FAR-"
- board text removed: "+RED-"

Commit message: Syncing AISLER project with GitHub repository
Parts:
- removed the REF** at (67.4, 96.2)
- removed the REF** at (62.3, 88.5)
- removed the REF** at (138.4, 110.4)
- added REF**: OSHW-Logo2_7.3x6mm_SilkScreen, Symbol:OSHW-Logo2_7.3x6mm_SilkScreen, F.Cu at (111.2, 68.5)
- added REF**: Shadock2, ressources:Shadock2_Cu, B.Cu at (105.5, 138.0)
- moved REF** 76.2 mm to (112.8, 63.5), turned to 0 degrees
- moved REF** 57.6 mm to (63.5, 93.5)
- moved REF** 1.99 mm to (96.2, 59.8)
- moved REF** 0.70 mm to (64.5, 122.0)
Routing:
- net GND: vias 12 -> 0
- removed copper zone on B.Cu, net GND
Other:
- board text added: "AstroPlant LED pannel Proto MK0.2 Vincent Frangi"
- board text removed: "AstroPlant LED Proto MK0.2 Vincent Frangi"
- board text removed: "Quand on ne sait pas où l'on va, il faut y aller !!... ...Et le plus vite possible."

Commit message: Syncing AISLER project with GitHub repository
Parts:
- removed the G*** at (106.0, 77.8)
- removed the G*** at (136.0, 90.8)
- removed the REF** at (112.8, 63.5)
- removed the REF** at (96.2, 59.8)
- removed the REF** at (64.5, 122.0)
- removed the REF** at (105.5, 138.0)
- REF**: moved to F.Cu
- moved REF** 36.6 mm to (99.5, 100.2)
Routing:
- net THERMAL_PAD: vias 125 -> 0
- removed copper zone on B.Cu, net THERMAL_PAD
- removed copper zone on F.Cu, net THERMAL_PAD
Other:
- board text added: "AstroPlant LED pannel Proto MK0.1 Vincent Frangi"
- board text removed: "AstroPlant LED pannel Proto MK0.2 Vincent Frangi"
- board text removed: "Shadoks Edition"
